Commit message: [mod]lrf collision position

File: rab_description/urdf/sensors/lrf/lrf.urdf.xacro (robot description, xacro)
@@ -16,4 +16,5 @@
       </visual>
       <collision>
+      <origin xyz="0 0 -0.055"/>
         <geometry>
 	  <mesh filename="package://rab_description/meshes/STL/${prefix}_lrf_link.stl"/>
