Commit message: [mod]provisional

File: rab_description/urdf/base/base.urdf.xacro (robot description, xacro)
@@ -20,8 +20,8 @@
 	    </collision>
 	    <inertial>
-	        <origin xyz="0 0 0.11" />
-		<mass value="20.0" />
-		<inertia ixx="2.2230" ixy="0" ixz="0"
-		         iyy="3.3236" iyz="0" izz="2.5307"/>
+	        <origin xyz="0 0 0" />
+		<mass value="20.598" />
+		<inertia ixx="2.708" ixy="0" ixz="0"
+		         iyy="5.185" iyz="0" izz="3.383"/>
 	    </inertial>
 	 </link>

File: rab_description/urdf/wheel/wheel.urdf.xacro (robot description, xacro)
@@ -6,5 +6,5 @@
    <property name="wheel_radius" value="0.110"/>
    <property name="wheel_length" value="0.045"/>
-   <property name="wheel_mass" value="1.0" />
+   <property name="wheel_mass" value="1.832" />
    <xacro:macro name="wheel_v0" params="prefix parent *joint_origin *joint_axis">
          <joint name="${prefix}_wheel_joint" type="continuous">
@@ -21,5 +21,5 @@
 	    </visual>
 	    <collision>
-	       <origin xyz="0 -0.003 0" rpy="${-M_PI/2} 0 0"/>
+	       <origin xyz="0 0 0" rpy="${-M_PI/2} 0 0"/>
  	       <geometry>
 	          <cylinder radius="${wheel_radius}" length="${wheel_length}"/>
@@ -27,5 +27,5 @@
 	    </collision>
 	    <inertial>
-	       <origin xyz="0 -0.003 0" rpy="${M_PI/2} 0 0"/>
+	       <origin xyz="0 0 0" rpy="${M_PI/2} 0 0"/>
 	       <cylinder_inertial mass="${wheel_mass}"
                                   radius="${wheel_radius}" length="${wheel_length}"/>

Commit message: [mod]inertia

File: rab_description/urdf/base/base.urdf.xacro (robot description, xacro)
@@ -21,7 +21,7 @@
 	    <inertial>
 	        <origin xyz="0 0 0" />
-		<mass value="25.897" />
-		<inertia ixx="1.772" ixy="0" ixz="0"
-		         iyy="3.35" iyz="0" izz="2.269"/>
+		<mass value="20.0" />
+		<inertia ixx="1.9333" ixy="0" ixz="0"
+		         iyy="3.3333" iyz="0" izz="1.93333"/>
 	    </inertial>
 	 </link>

File: rab_description/urdf/wheel/wheel.urdf.xacro (robot description, xacro)
@@ -6,5 +6,5 @@
    <property name="wheel_radius" value="0.110"/>
    <property name="wheel_length" value="0.045"/>
-   <property name="wheel_mass" value="1.832" />
+   <property name="wheel_mass" value="1.8" />
    <xacro:macro name="wheel_v0" params="prefix parent *joint_origin *joint_axis">
          <joint name="${prefix}_wheel_joint" type="continuous">

Commit message: [mod]inertial

File: rab_description/urdf/base/base.urdf.xacro (robot description, xacro)
@@ -20,8 +20,8 @@
 	    </collision>
 	    <inertial>
-	        <origin xyz="0 0 0" />
-		<mass value="20.0" />
-		<inertia ixx="1.9333" ixy="0" ixz="0"
-		         iyy="3.3333" iyz="0" izz="1.93333"/>
+	        <origin xyz="0.39 0 0.13" />
+		<mass value="21.505" />
+		<inertia ixx="1.338" ixy="0" ixz="0"
+		         iyy="3.407" iyz="0" izz="2.634"/>
 	    </inertial>
 	 </link>
