Commit message: [mod]lrf_position

File: rab_description/robots/rab.urdf.xacro (robot description, xacro)
@@ -24,9 +24,9 @@
    <!-- right_lrf -->
    <xacro:lrf_v0 prefix="right" parent="base_link">
-         <origin xyz="-0.032 -0.246 0.137" rpy="0 0 -1.57" />
+         <origin xyz="-0.032 -0.246 0.185" rpy="0 0 -1.57" />
    </xacro:lrf_v0>
    <!-- left_lrf -->
    <xacro:lrf_v0 prefix="left" parent="base_link">
-         <origin xyz="-0.032 0.246 0.137" rpy="0 0 1.57" />
+         <origin xyz="-0.032 0.246 0.185" rpy="0 0 1.57" />
    </xacro:lrf_v0>
    <link name="lrf_link"/>

File: rab_description/urdf/base/base.urdf.xacro (robot description, xacro)
@@ -21,7 +21,7 @@
 	    <inertial>
 	        <origin xyz="0 0 0" />
-		<mass value="20.598" />
-		<inertia ixx="2.708" ixy="0" ixz="0"
-		         iyy="5.185" iyz="0" izz="3.383"/>
+		<mass value="25.897" />
+		<inertia ixx="1.772" ixy="0" ixz="0"
+		         iyy="3.35" iyz="0" izz="2.269"/>
 	    </inertial>
 	 </link>

File: rab_description/urdf/sensors/lrf/lrf.urdf.xacro (robot description, xacro)
@@ -21,5 +21,5 @@
       </collision>
       <inertial>
-        <origin xyz="0 0 -0.0164"/>
+        <origin xyz="0 0 0"/>
 	<box_inertial mass="0.4" height="0.07" width="0.07" depth="0.08"/>
       </inertial>

Commit message: [mod]wheel_link position

File: rab_description/robots/rab.urdf.xacro (robot description, xacro)
@@ -13,10 +13,10 @@
    <!-- right_wheel -->
    <xacro:wheel_v0 prefix="right" parent="base_link">
-         <origin xyz="0 -0.265 0"/>
+         <origin xyz="0 -0.262 0"/>
 	 <axis xyz="0 1 0"/>
    </xacro:wheel_v0>
    <!-- left_wheel -->
    <xacro:wheel_v0 prefix="left" parent="base_link">
-         <origin xyz="0 0.265 0"/>
+         <origin xyz="0 0.262 0" rpy="0 0 -${M_PI}"/>
 	 <axis xyz="0 -1 0"/>
    </xacro:wheel_v0>

Commit message: [add]3d_sensor

File: rab_description/robots/rab.urdf.xacro (robot description, xacro)
@@ -36,4 +36,10 @@
 	 <origin xyz="-0.032 0 0.137"/>
    </joint>
+   <link name="3d_sensor_link"/>
+   <joint name="3d_sensor_link_joint" type="fixed">
+         <parent link="base_link"/>
+	 <child link="3d_sensor_link"/>
+	 <origin xyz="0.59 0 0.265"/>
+   </joint>
    <!-- =========== transmission ============= -->
    <xacro:wheel_trans_v0 prefix="right"/>
